Commit message: fixed imu

File: src/rover_description/urdf/gazebo.urdf.xacro (robot description, xacro)
@@ -134,5 +134,5 @@
       </plugin>
       <plugin filename="ignition-gazebo-sensors-system" name="ignition::gazebo::systems::Sensors">
-        <render_engine>ogre2</render_engine>
+        <!-- <render_engine>ogre2</render_engine> -->
       </plugin>
     </xacro:if>
@@ -145,32 +145,58 @@
       </plugin>
       <plugin filename="gz-sim-sensors-system" name="gz::sim::systems::Sensors">
-        <render_engine>ogre2</render_engine>
+        <!-- <render_engine>ogre2</render_engine> -->
       </plugin>
     </xacro:unless>
   </gazebo>
-  <!-- <gazebo>
-    <plugin filename="libgazebo_ros2_control.so" name="gazebo_ros2_control">
-      <parameters>$(find rover_controller)/config/controller_velocity.yaml</parameters>
-    </plugin>
-  </gazebo> -->
+  <!-- IMU -->
   <gazebo reference="imu_link">
-      <gravity>true</gravity>
-      <sensor name="imu_sensor" type="imu">
-      <always_on>true</always_on>
-      <update_rate>100</update_rate>
-      <visualize>true</visualize>
-      <topic>"imu"</topic>
-      <plugin filename="libgazebo_ros_imu_sensor.so" name="imu_plugin">
-          <topicName>imu</topicName>
-          <bodyName>imu_link</bodyName>
-          <updateRateHZ>100.0</updateRateHZ>
-          <gaussianNoise>0.0</gaussianNoise>
-          <xyzOffset>0 0 0</xyzOffset>
-          <rpyOffset>0 0 0</rpyOffset>
-          <frameName>imu_link</frameName>
-          <initialOrientationAsReference>false</initialOrientationAsReference>
-      </plugin>
-      <pose>0 0 0 0 0 0</pose>
-      </sensor>
+    <sensor name="imu" type="imu">
+        <always_on>true</always_on>
+        <update_rate>100</update_rate>
+        <gz_frame_id>imu_link</gz_frame_id>
+        <topic>imu</topic>
+        <imu>
+          <angular_velocity>
+            <x>
+              <noise type="gaussian">
+                <mean>0.0</mean>
+                <stddev>2e-4</stddev>
+              </noise>
+            </x>
+            <y>
+              <noise type="gaussian">
+                <mean>0.0</mean>
+                <stddev>2e-4</stddev>
+              </noise>
+            </y>
+            <z>
+              <noise type="gaussian">
+                <mean>0.0</mean>
+                <stddev>2e-4</stddev>
+              </noise>
+            </z>
+          </angular_velocity>
+          <linear_acceleration>
+            <x>
+              <noise type="gaussian">
+                <mean>0.0</mean>
+                <stddev>1.7e-2</stddev>
+              </noise>
+            </x>
+            <y>
+              <noise type="gaussian">
+                <mean>0.0</mean>
+                <stddev>1.7e-2</stddev>
+              </noise>
+            </y>
+            <z>
+              <noise type="gaussian">
+                <mean>0.0</mean>
+                <stddev>1.7e-2</stddev>
+              </noise>
+            </z>
+          </linear_acceleration>
+        </imu>
+    </sensor>
   </gazebo>
   <!-- 2D Laser Sensor -->
@@ -202,11 +228,4 @@
         </noise>
       </lidar>
-      <!-- <plugin name="laser_controller" filename="libgazebo_ros_ray_sensor.so">
-          <ros>
-              <argument>~/out:=scan</argument>
-          </ros>
-          <output_type>sensor_msgs/LaserScan</output_type>
-          <frame_name>laser_link</frame_name>
-      </plugin> -->
     </sensor>
   </gazebo>

File: src/rover_description/urdf/osr.urdf.xacro (robot description, xacro)
@@ -418,10 +418,32 @@
     <xacro:wheel prefix="left" dir="1" origin="0" prefix_1="L"/>
     <xacro:wheel prefix="right" dir="-1" origin="3.14" prefix_1="R"/>
-    <joint name="imu_joint" type="fixed">
-            <parent link="base_link"/>
-            <child link="imu_link"/>
-            <origin xyz="0 0 0" rpy="0 0 0"/>
-        </joint>
-    <link name="imu_link"></link>
+    <link name="imu_link">
+        <inertial>
+          <origin xyz="-0.00552433659106688 0.000168210391520346 0.000514000497342681" rpy="0 0 0" />
+          <mass value="0.000528415362211671" />
+          <inertia ixx="1.46176048428261E-08" ixy="1.40015117949421E-10" ixz="-1.99633872937403E-12"
+                   iyy="8.59662482954888E-09" iyz="7.52375112767959E-12"
+                   izz="2.30279421279312E-08" />
+        </inertial>
+        <visual>
+          <origin xyz="0 0 0" rpy="0 0 0" />
+          <geometry>
+            <mesh filename="package://bumperbot_description/meshes/imu_link.STL" />
+          </geometry>
+          <material name="blue"/>
+        </visual>
+        <collision>
+          <origin xyz="0 0 0" rpy="0 0 0" />
+          <geometry>
+            <mesh filename="package://bumperbot_description/meshes/imu_link.STL" />
+          </geometry>
+        </collision>
+      </link>
+      <joint name="imu_joint" type="fixed">
+        <origin xyz="0 0 0.0698986241758014" rpy="0 0 0" />
+        <parent link="base_link" />
+        <child link="imu_link" />
+        <axis xyz="0 0 0" />
+      </joint>
     <link name="laser_link">
         <inertial>
