Commit message: added navigation, not working

File: src/rover_description/urdf/osr.urdf.xacro (robot description, xacro)
@@ -429,5 +429,5 @@
           <origin xyz="0 0 0" rpy="0 0 0" />
           <geometry>
-            <mesh filename="package://bumperbot_description/meshes/imu_link.STL" />
+            <mesh filename="package://rover_description/meshes/imu_link.STL" />
           </geometry>
           <material name="blue"/>
@@ -436,5 +436,5 @@
           <origin xyz="0 0 0" rpy="0 0 0" />
           <geometry>
-            <mesh filename="package://bumperbot_description/meshes/imu_link.STL" />
+            <mesh filename="package://rover_description/meshes/imu_link.STL" />
           </geometry>
         </collision> -->
