Commit message: simple controller code organize

File: install/rover_description/share/rover_description/urdf/osr.urdf.xacro (robot description, xacro)
@@ -419,5 +419,5 @@
     <xacro:wheel prefix="right" dir="-1" origin="3.14" prefix_1="R"/>
     <link name="imu_link">
-        <inertial>
+        <!-- <inertial>
           <origin xyz="-0.00552433659106688 0.000168210391520346 0.000514000497342681" rpy="0 0 0" />
           <mass value="0.000528415362211671" />
@@ -438,5 +438,5 @@
             <mesh filename="package://bumperbot_description/meshes/imu_link.STL" />
           </geometry>
-        </collision>
+        </collision> -->
       </link>
       <joint name="imu_joint" type="fixed">
