Commit message: fixed odom problem

File: install/rover_description/share/rover_description/urdf/gazebo.urdf.xacro (robot description, xacro)
@@ -18,4 +18,22 @@
         </xacro:unless>
     </xacro:if>
+    <joint name="front_wheel_joint_left">
+      <command_interface name="velocity">
+        <param name="min">-10</param>
+        <param name="max">10</param>
+      </command_interface>
+      <state_interface name="position"/>
+      <state_interface name="velocity"/>
+      <state_interface name="effort"/>
+    </joint>
+    <joint name="front_wheel_joint_right">
+      <command_interface name="velocity">
+        <param name="min">-10</param>
+        <param name="max">10</param>
+      </command_interface>
+      <state_interface name="position"/>
+      <state_interface name="velocity"/>
+      <state_interface name="effort"/>
+    </joint>
     <joint name="middle_wheel_joint_left">
       <command_interface name="velocity">
@@ -25,4 +43,5 @@
       <state_interface name="position"/>
       <state_interface name="velocity"/>
+      <state_interface name="effort"/>
     </joint>
     <joint name="middle_wheel_joint_right">
@@ -53,17 +72,12 @@
       <state_interface name="effort"/>
     </joint>
-    <joint name="front_wheel_joint_left">
-      <command_interface name="velocity">
-        <param name="min">-10</param>
-        <param name="max">10</param>
-      </command_interface>
-      <state_interface name="position"/>
-      <state_interface name="velocity"/>
-      <state_interface name="effort"/>
-    </joint>
-    <joint name="front_wheel_joint_right">
-      <command_interface name="velocity">
-        <param name="min">-10</param>
-        <param name="max">10</param>
+    <joint name="front_wheel_joint_L">
+      <command_interface name="position">
+        <param name="min">-5</param>
+        <param name="max">5</param>
+      </command_interface>
+      <command_interface name="velocity">
+        <param name="min">-0.1</param>
+        <param name="max">0.1</param>
       </command_interface>
       <state_interface name="position"/>
@@ -84,5 +98,5 @@
       <state_interface name="effort"/>
     </joint>
-    <joint name="front_wheel_joint_L">
+    <joint name="rear_wheel_joint_L">
       <command_interface name="position">
         <param name="min">-5</param>
@@ -98,17 +112,4 @@
     </joint>
     <joint name="rear_wheel_joint_R">
-      <command_interface name="position">
-        <param name="min">-5</param>
-        <param name="max">5</param>
-      </command_interface>
-      <command_interface name="velocity">
-        <param name="min">-0.1</param>
-        <param name="max">0.1</param>
-      </command_interface>
-      <state_interface name="position"/>
-      <state_interface name="velocity"/>
-      <state_interface name="effort"/>
-    </joint>
-    <joint name="rear_wheel_joint_L">
       <command_interface name="position">
         <param name="min">-5</param>
